File: lcd.kicad_sch (KiCad schematic)
At the start: 2 parts

Commit message: Add files via upload
Changed lines of the file:
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@@
       (effects (font (size 1.27 1.27)) hide)
     )
-    (property "Value" "" (id 1) (at 125.73 78.867 0))
+    (property "Value" "VCC" (id 1) (at 125.73 78.867 0))
     (property "Footprint" "" (id 2) (at 125.73 84.074 0)
       (effects (font (size 1.27 1.27)) hide)
