File: 280F10_CMOSFlash.kicad_sch (KiCad schematic)
At the start: 3 parts

Commit message: Add files via upload
Parts:
- U?: value (none) -> PAL16L8; footprint (none) -> Package_DIP:DIP-20_W7.62mm
- U? (x2): value (none) -> 28F010; footprint (none) -> 28F010
Connections:
- net A10: now also U?.23 (A10)
- net GND: now also U?.16 (VSS), U?.16 (VSS)
- net VCC: now also U?.1 (VPP), U?.1 (VPP), U?.32 (VCC), U?.32 (VCC)
- net D0: now reaches U?.13 (DQ0)
- net D0: now also U?.13 (DQ0)
- net D1: now reaches U?.14 (DQ1)
- net D1: now also U?.14 (DQ1)
- net D2: now reaches U?.15 (DQ2)
- net D2: now also U?.15 (DQ2)
- net D3: now reaches U?.17 (DQ3)
- net D3: now also U?.17 (DQ3)
- net D4: now reaches U?.18 (DQ4)
- net D4: now also U?.18 (DQ4)
- net D5: now reaches U?.19 (DQ5)
- net D5: now also U?.19 (DQ5)
- net D6: now reaches U?.20 (DQ6)
- net D6: now also U?.20 (DQ6)
- net D7: now reaches U?.21 (DQ7)
- net D7: now also U?.21 (DQ7)
- net AD18 renamed A18
- net AD19 renamed A19

Commit message: Add files via upload
Connections:
- net A0 is gone; now on net A19: U?.12 (A0), U?.12 (A0), U?.3 (A0)
- net VCC: no longer U?.1 (VPP), U?.32 (VCC)
- new net: U?.1 (VPP), U?.32 (VCC)
Other:
- moved on the sheet: U?
