File: CY7C199_SRAM.kicad_sch (KiCad schematic)
At the start: 5 parts

Commit message: Add files via upload
Parts:
- U? (x4): value (none) -> CY7C199
Connections:
- net at U?.19 (IO1): now also U?.20 (~{CE}), U?.22 (~{OE})
- net at U?.14 (GND): now also U?.14 (GND)
- new net: U?.14 (GND), U?.14 (GND)

Commit message: Add files via upload
Connections:
- net A0: no longer U?.21 (A0)
- net A1: no longer U?.23 (A1)
- net A10: no longer U?.6 (A10)
- net A11: no longer U?.7 (A11)
- net A12: no longer U?.8 (A12)
- net A13: no longer U?.9 (A13)
- net A14: no longer U?.10 (A14)
- net A2: no longer U?.24 (A2)
- net A3: no longer U?.25 (A3)
- net A4: no longer U?.26 (A4)
- net A5: no longer U?.1 (A5)
- net A6: no longer U?.2 (A6)
- net A7: no longer U?.3 (A7)
- net A8: no longer U?.4 (A8)
- net A9: no longer U?.5 (A9)
