File: finalproj.kicad_sch (KiCad schematic)
At the start: 33 parts, among them J1 Conn_01x16, SW1 SW_Push, U1 8284, U10 CY7C199, U11 CY7C199, U2 8086_Min_Mode, U5 PAL16L8, U7 CY7C199, U8 CY7C199, U9 PAL16L8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

Commit message: Add files via upload
Parts:
- removed C? (x6): C, symbol Device:C
- removed C?: (no value), symbol Device:C
- removed J1: Conn_01x16, Connector_JST:JST_PH_B16B-PH-K_1x16_P2.00mm_Vertical, symbol Connector_Generic:Conn_01x16
- removed J?: (no value), symbol Connector:DB9_Female
- removed R?: R, symbol Device:R
- removed R? (x2): (no value), symbol Device:R
- removed R?: R, OptoDevice:R_LDR_4.9x4.2mm_P2.54mm_Vertical, symbol Device:R
- removed U10, U11, U7, U8: CY7C199, symbol Memory_RAM:CY7C199
- removed U5: PAL16L8, Package_DIP:DIP-20_W7.62mm, symbol Logic_Programmable:PAL16L8
- removed U9, U?: PAL16L8, symbol Logic_Programmable:PAL16L8
- removed U? (x2): 28F010, 28F010, symbol 28F010:28F010
- removed U?: (no value), symbol Display_Character:NHD-0420H1Z
- removed U?: 16550, Package_DIP:DIP-40_W15.24mm, symbol Interface_UART:16550
- removed U?: max235cpg, max235cpg, symbol max235cpg:max235cpg
- removed U?: MAX232, symbol Interface_UART:MAX232
- removed Y?: Crystal, Crystal:Crystal_AT310_D3.0mm_L10.0mm_Horizontal, symbol Device:Crystal
- added J?: (no value), symbol Connector:Conn_01x03_Male
- added J?: Conn_01x08_Male, symbol Connector:Conn_01x08_Male
- added J?: (no value), symbol Connector:Conn_01x04_Male
- added J?: (no value), symbol Connector:Conn_01x08_Male
Connections:
- net AD6: now reaches U2.10 (AD6)
- net AD5: now reaches U2.11 (AD5)
- net AD4: now reaches U2.12 (AD4)
- net AD3: now reaches U2.13 (AD3)
- net AD2: now reaches U2.14 (AD2)
- net AD1: now reaches U2.15 (AD1)
- net AD0: now reaches U2.16 (AD0)
- net INTR: now reaches U2.18 (INTR)
- net CLK: now reaches U1.8 (CLK), U2.19 (CLK)
- net AD14: now reaches U2.2 (AD14)
- net RESET: now reaches U1.5 (READY), U2.22 (READY)
- net AD13: now reaches U2.3 (AD13)
- net BHE: now reaches U2.34 (~{BHE}/S7)
- net A19: now reaches U2.35 (A19/S6)
- net A18: now reaches U2.36 (A18/S5)
- net A17: now reaches U2.37 (A17/S4)
- net A16: now reaches U2.38 (A16/S3)
- net AD12: now reaches U2.4 (AD12)
- net AD9: now reaches U2.7 (AD9)
- net AD8: now reaches U2.8 (AD8)
- net AD7: now reaches U2.9 (AD7)
Other:
- added sheet 28F010 CMOS Flash (280F10_CMOSFlash.kicad_sch)
- added sheet CY7C199 SRAM (CY7C199_SRAM.kicad_sch)
- added sheet LCD (lcd.kicad_sch)
- added sheet UART (uart.kicad_sch)
- moved on the sheet: 10e-6F1, 10kohm1, SW1, U1, U2, Y1

Commit message: Add files via upload
Parts:
- added J?: (no value), symbol Connector:Conn_01x09_Male
- J?: value (none) -> Conn_01x03_Male
- J?: value (none) -> Conn_01x04_Male
- J?: value (none) -> Conn_01x08_Male
Connections:
- net GND: now also U2.1 (GND), U2.20 (GND)
- net INTA: now reaches U2.24 (~{INTA})
- net A15: now reaches U2.39 (AD15)
- net A11: now reaches U2.5 (AD11)
- net A10: now reaches U2.6 (AD10)
- net AD0 renamed A0
- net AD1 renamed A1
- net AD12 renamed A12
- net AD13 renamed A13
- net AD14 renamed A14
- net AD2 renamed A2
- net AD3 renamed A3
- net AD4 renamed A4
- net AD5 renamed A5
- net AD6 renamed A6
- net AD7 renamed A7
- net AD8 renamed A8
- net AD9 renamed A9
Other:
- added sheet switches (switches.kicad_sch)
- moved on the sheet: J?

Commit message: Add files via upload
Parts:
- J?: value (none) -> Conn_01x09_Male
Other:
- sheet UART ports: added A0, A1, A2; removed none
Changed lines of the file:
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@@
       (effects (font (size 1.27 1.27)) hide)
     )
-    (property "Value" "" (id 1) (at 221.361 131.445 0))
+    (property "Value" "GND" (id 1) (at 221.361 131.445 0))
     (property "Footprint" "" (id 2) (at 221.361 126.873 0)
       (effects (font (size 1.27 1.27)) hide)
@@
     (in_bom yes) (on_board yes) (fields_autoplaced)
     (property "Reference" "J?" (id 0) (at 172.466 117.602 0))
-    (property "Value" "" (id 1) (at 172.466 120.142 0))
+    (property "Value" "Conn_01x09_Male" (id 1) (at 172.466 120.142 0))
     (property "Footprint" "" (id 2) (at 171.831 132.969 0)
       (effects (font (size 1.27 1.27)) hide)
@@
       (effects (font (size 1.27 1.27)) (justify left top))
     )
-  )
+    (pin "A1" bidirectional (at 54.61 69.723 180)
+      (effects (font (size 1.27 1.27)) (justify left))
+    )
+    (pin "A2" bidirectional (at 54.61 72.644 180)
+      (effects (font (size 1.27 1.27)) (justify left))
+    )
+    (pin "A0" bidirectional (at 54.61 66.929 180)
+      (effects (font (size 1.27 1.27)) (justify left))
+    )
+  )
