File: switches.kicad_sch (KiCad schematic)
At the start: 12 parts

Commit message: Add files via upload
Parts:
- R?: value (none) -> R
- SW?: value (none) -> SW_DIP_x08
- U?: value (none) -> 74LVC1G11
- U?: value (none) -> 74LS540
Changed lines of the file:
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@@
       (effects (font (size 1.27 1.27)) hide)
     )
-    (property "Value" "" (id 1) (at 117.475 110.617 0))
+    (property "Value" "GND" (id 1) (at 117.475 110.617 0))
     (property "Footprint" "" (id 2) (at 117.475 105.791 0)
       (effects (font (size 1.27 1.27)) hide)
@@
       (effects (font (size 1.27 1.27)) (justify left))
     )
-    (property "Value" "" (id 1) (at 78.74 64.1349 0)
+    (property "Value" "R" (id 1) (at 78.74 64.1349 0)
       (effects (font (size 1.27 1.27)) (justify left))
     )
@@
       (effects (font (size 1.27 1.27)) hide)
     )
-    (property "Value" "" (id 1) (at 88.773 87.63 0))
+    (property "Value" "VCC" (id 1) (at 88.773 87.63 0))
     (property "Footprint" "" (id 2) (at 88.773 92.837 0)
       (effects (font (size 1.27 1.27)) hide)
@@
     (in_bom yes) (on_board yes) (fields_autoplaced)
     (property "Reference" "U?" (id 0) (at 66.2305 90.17 0))
-    (property "Value" "" (id 1) (at 66.2305 92.71 0))
+    (property "Value" "74LVC1G11" (id 1) (at 66.2305 92.71 0))
     (property "Footprint" "" (id 2) (at 66.548 98.933 0)
       (effects (font (size 1.27 1.27)) hide)
@@
       (effects (font (size 1.27 1.27)) hide)
     )
-    (property "Value" "" (id 1) (at 117.475 57.15 0))
+    (property "Value" "VCC" (id 1) (at 117.475 57.15 0))
     (property "Footprint" "" (id 2) (at 117.475 62.23 0)
       (effects (font (size 1.27 1.27)) hide)
@@
       (effects (font (size 1.27 1.27)) hide)
     )
-    (property "Value" "" (id 1) (at 55.499 80.0099 90)
+    (property "Value" "GND" (id 1) (at 55.499 80.0099 90)
       (effects (font (size 1.27 1.27)) (justify right))
     )
@@
       (effects (font (size 1.27 1.27)) hide)
     )
-    (property "Value" "" (id 1) (at 92.583 53.34 0))
+    (property "Value" "VCC" (id 1) (at 92.583 53.34 0))
     (property "Footprint" "" (id 2) (at 92.583 58.166 0)
       (effects (font (size 1.27 1.27)) hide)
@@
       (effects (font (size 1.27 1.27)) (justify left))
     )
-    (property "Value" "" (id 1) (at 119.4944 65.913 0)
+    (property "Value" "74LS540" (id 1) (at 119.4944 65.913 0)
       (effects (font (size 1.27 1.27)) (justify left))
     )
@@
     (in_bom yes) (on_board yes) (fields_autoplaced)
     (property "Reference" "SW?" (id 0) (at 70.104 63.5 0))
-    (property "Value" "" (id 1) (at 70.104 66.04 0))
+    (property "Value" "SW_DIP_x08" (id 1) (at 70.104 66.04 0))
     (property "Footprint" "" (id 2) (at 70.104 81.153 0)
       (effects (font (size 1.27 1.27)) hide)
@@
       (effects (font (size 1.27 1.27)) hide)
     )
-    (property "Value" "" (id 1) (at 88.773 133.604 0))
+    (property "Value" "GND" (id 1) (at 88.773 133.604 0))
     (property "Footprint" "" (id 2) (at 88.773 128.143 0)
       (effects (font (size 1.27 1.27)) hide)
