File: uart.kicad_sch (KiCad schematic)
At the start: 16 parts

Commit message: Add files via upload
Parts:
- added U?: 4081, symbol 4xxx:4081
Connections:
- net GND: now also U?.20 (GND)
- net AD1 renamed A1
- net AD15-AD5: no longer names the net of U?.1 (A15-A5)
- net AD15-AD5: now also U?.5
- net AD4 renamed A4
- new net A15-A8: U?.1
- new net A5: U?.2
- new net A6: U?.4
- new net A7: U?.3
Changed lines of the file:
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@@
+    (stroke (width 0) (type default) (color 0 0 0 0))
+  )
+  (wire (pts (xy 30.988 91.948) (xy 32.004 91.948))
     (stroke (width 0) (type default) (color 0 0 0 0))
   )
@@
     (stroke (width 0) (type default) (color 0 0 0 0))
   )
-  (wire (pts (xy 107.823 126.492) (xy 110.49 126.492))
+  (wire (pts (xy 106.172 126.492) (xy 110.49 126.492))
+    (stroke (width 0) (type default) (color 0 0 0 0))
+  )
+  (wire (pts (xy 107.95 129.032) (xy 107.95 129.413))
     (stroke (width 0) (type default) (color 0 0 0 0))
   )
@@
     (stroke (width 0) (type default) (color 0 0 0 0))
   )
+  (wire (pts (xy 135.89 136.652) (xy 135.89 137.922))
+    (stroke (width 0) (type default) (color 0 0 0 0))
+  )
   (wire (pts (xy 107.696 118.872) (xy 107.696 116.332))
     (stroke (width 0) (type default) (color 0 0 0 0))
@@
     (stroke (width 0) (type default) (color 0 0 0 0))
   )
+  (wire (pts (xy 30.988 89.408) (xy 32.004 89.408))
+    (stroke (width 0) (type default) (color 0 0 0 0))
+  )
   (wire (pts (xy 47.371 95.758) (xy 49.784 95.758))
     (stroke (width 0) (type default) (color 0 0 0 0))
@@
     (stroke (width 0) (type default) (color 0 0 0 0))
   )
+  (wire (pts (xy 30.988 94.488) (xy 32.004 94.488))
+    (stroke (width 0) (type default) (color 0 0 0 0))
+  )
   (wire (pts (xy 135.89 50.038) (xy 164.846 50.038))
     (stroke (width 0) (type default) (color 0 0 0 0))
@@
     (stroke (width 0) (type default) (color 0 0 0 0))
   )
+  (wire (pts (xy 107.95 129.413) (xy 106.172 129.413))
+    (stroke (width 0) (type default) (color 0 0 0 0))
+  )
   (wire (pts (xy 165.608 98.552) (xy 165.608 112.522))
     (stroke (width 0) (type default) (color 0 0 0 0))
@@
     (stroke (width 0) (type default) (color 0 0 0 0))
   )
+  (wire (pts (xy 30.988 86.868) (xy 32.004 86.868))
+    (stroke (width 0) (type default) (color 0 0 0 0))
+  )
   (wire (pts (xy 108.204 60.452) (xy 108.204 60.198))
     (stroke (width 0) (type default) (color 0 0 0 0))
@@
   (wire (pts (xy 105.918 121.666) (xy 110.49 121.666))
     (stroke (width 0) (type default) (color 0 0 0 0))
+  )
+  (global_label "RESET" (shape output) (at 106.172 129.413 180) (fields_autoplaced)
+    (effects (font (size 1.27 1.27)) (justify right))
+    (property "Intersheet References" "${INTERSHEET_REFS}" (id 0) (at 98.0137 129.4924 0)
+      (effects (font (size 1.27 1.27)) (justify right) hide)
+    )
+  )
+  (global_label "INTR" (shape output) (at 106.172 126.492 180) (fields_autoplaced)
+    (effects (font (size 1.27 1.27)) (justify right))
+    (property "Intersheet References" "${INTERSHEET_REFS}" (id 0) (at 99.586 126.4126 0)
+      (effects (font (size 1.27 1.27)) (justify right) hide)
+    )
   )
   (global_label "D0-D7" (shape bidirectional) (at 105.664 56.515 0) (fields_autoplaced)
@@
     )
   )
+  (hierarchical_label "A15-A8" (shape input) (at 30.988 86.868 180)
+    (effects (font (size 1.27 1.27)) (justify right))
+  )
+  (hierarchical_label "A7" (shape input) (at 30.988 89.408 180)
+    (effects (font (size 1.27 1.27)) (justify right))
+  )
   (hierarchical_label "TXRDY" (shape output) (at 162.814 111.252 0)
     (effects (font (size 1.27 1.27)) (justify left))
   )
+  (hierarchical_label "A5" (shape input) (at 30.988 94.488 180)
+    (effects (font (size 1.27 1.27)) (justify right))
+  )
   (hierarchical_label "RD" (shape input) (at 105.918 121.666 180)
-    (effects (font (size 1.27 1.27)) (justify right))
-  )
-  (hierarchical_label "INTR" (shape output) (at 107.823 126.492 180)
     (effects (font (size 1.27 1.27)) (justify right))
   )
@@
     (effects (font (size 1.27 1.27)) (justify left))
   )
-  (hierarchical_label "RESET" (shape input) (at 107.95 129.032 180)
-    (effects (font (size 1.27 1.27)) (justify right))
-  )
   (hierarchical_label "WR" (shape input) (at 107.569 113.792 180)
     (effects (font (size 1.27 1.27)) (justify right))
@@
     (effects (font (size 1.27 1.27)) (justify left))
   )
-  (hierarchical_label "AD1" (shape input) (at 108.077 83.312 180)
-    (effects (font (size 1.27 1.27)) (justify right))
-  )
-  (hierarchical_label "AD15-AD5" (shape input) (at 47.244 90.678 180)
-    (effects (font (size 1.27 1.27)) (justify right))
-  )
-  (hierarchical_label "AD2" (shape input) (at 108.204 85.852 180)
+  (hierarchical_label "A1" (shape bidirectional) (at 108.077 83.312 180)
+    (effects (font (size 1.27 1.27)) (justify right))
+  )
+  (hierarchical_label "A2" (shape bidirectional) (at 108.204 85.852 180)
     (effects (font (size 1.27 1.27)) (justify right))
   )
@@
     (effects (font (size 1.27 1.27)) (justify left))
   )
-  (hierarchical_label "AD4" (shape input) (at 47.371 93.218 180)
-    (effects (font (size 1.27 1.27)) (justify right))
-  )
-  (hierarchical_label "AD1" (shape input) (at 47.371 95.631 180)
-    (effects (font (size 1.27 1.27)) (justify right))
-  )
-  (hierarchical_label "AD0" (shape input) (at 108.077 80.899 180)
+  (hierarchical_label "A4" (shape input) (at 47.371 93.218 180)
+    (effects (font (size 1.27 1.27)) (justify right))
+  )
+  (hierarchical_label "A1" (shape input) (at 47.371 95.631 180)
+    (effects (font (size 1.27 1.27)) (justify right))
+  )
+  (hierarchical_label "A6" (shape input) (at 30.988 91.948 180)
+    (effects (font (size 1.27 1.27)) (justify right))
+  )
+  (hierarchical_label "A0" (shape bidirectional) (at 108.077 80.899 180)
     (effects (font (size 1.27 1.27)) (justify right))
   )
@@
     (pin "2")
   )
+  (symbol (lib_id "power:GND") (at 135.89 137.922 0) (unit 1)
+    (in_bom yes) (on_board yes) (fields_autoplaced)
+    (property "Reference" "#PWR?" (id 0) (at 135.89 144.272 0)
+      (effects (font (size 1.27 1.27)) hide)
+    )
+    (property "Value" "" (id 1) (at 135.89 143.51 0))
+    (property "Footprint" "" (id 2) (at 135.89 137.922 0)
+      (effects (font (size 1.27 1.27)) hide)
+    )
+    (property "Datasheet" "" (id 3) (at 135.89 137.922 0)
+      (effects (font (size 1.27 1.27)) hide)
+    )
+    (pin "1")
+  )
   (symbol (lib_id "power:VCC") (at 194.31 60.198 0) (unit 1)
     (in_bom yes) (on_board yes) (fields_autoplaced)
@@
       (effects (font (size 1.27 1.27)) hide)
     )
-    (property "Value" "" (id 1) (at 62.484 123.19 0))
+    (property "Value" "GND" (id 1) (at 62.484 123.19 0))
     (property "Footprint" "" (id 2) (at 62.484 118.618 0)
       (effects (font (size 1.27 1.27)) hide)
@@
       (effects (font (size 1.27 1.27)) hide)
     )
-    (property "Value" "" (id 1) (at 62.484 80.01 0))
+    (property "Value" "VCC" (id 1) (at 62.484 80.01 0))
     (property "Footprint" "" (id 2) (at 62.484 85.598 0)
       (effects (font (size 1.27 1.27)) hide)
@@
     (pin "1")
   )
+  (symbol (lib_id "4xxx:4081") (at 39.624 90.678 0) (unit 1)
+    (in_bom yes) (on_board yes) (fields_autoplaced)
+    (property "Reference" "U?" (id 0) (at 39.624 81.915 0))
+    (property "Value" "4081" (id 1) (at 39.624 84.455 0))
+    (property "Footprint" "" (id 2) (at 39.624 90.678 0)
+      (effects (font (size 1.27 1.27)) hide)
+    )
+    (property "Datasheet" "http://www.intersil.com/content/dam/Intersil/documents/cd40/cd4073bms-81bms-82bms.pdf" (id 3) (at 39.624 90.678 0)
+      (effects (font (size 1.27 1.27)) hide)
+    )
+    (pin "4")
+    (pin "1")
+    (pin "2")
+    (pin "3")
+    (pin "5")
+    (pin "4")
+    (pin "5")
+    (pin "6")
+    (pin "10")
+    (pin "8")
+    (pin "9")
+    (pin "11")
+    (pin "12")
+    (pin "13")
+    (pin "14")
+    (pin "7")
+  )
   (symbol (lib_id "Device:Crystal") (at 92.202 102.362 270) (unit 1)

Commit message: Add files via upload
Connections:
- net OUT1: no longer names the net of U?.34 (~{OUT1})
- net OUT2: no longer names the net of U?.31 (~{OUT2})
Changed lines of the file:
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@@
     (effects (font (size 1.27 1.27)) (justify right))
-  )
-  (hierarchical_label "OUT1" (shape output) (at 162.814 78.232 0)
-    (effects (font (size 1.27 1.27)) (justify left))
   )
   (hierarchical_label "A1" (shape bidirectional) (at 108.077 83.312 180)
@@
   (hierarchical_label "A2" (shape bidirectional) (at 108.204 85.852 180)
     (effects (font (size 1.27 1.27)) (justify right))
-  )
-  (hierarchical_label "OUT2" (shape output) (at 163.322 85.725 0)
-    (effects (font (size 1.27 1.27)) (justify left))
   )
   (hierarchical_label "A4" (shape input) (at 47.371 93.218 180)
@@
       (effects (font (size 1.27 1.27)) hide)
     )
-    (property "Value" "" (id 1) (at 135.89 143.51 0))
+    (property "Value" "GND" (id 1) (at 135.89 143.51 0))
     (property "Footprint" "" (id 2) (at 135.89 137.922 0)
       (effects (font (size 1.27 1.27)) hide)
@@
       (effects (font (size 1.27 1.27)) hide)
     )
+    (pin "1")
+    (pin "2")
+    (pin "3")
     (pin "4")
-    (pin "1")
-    (pin "2")
-    (pin "3")
     (pin "5")
     (pin "4")
