File: 8254.kicad_sch (KiCad schematic)
At the start: 2 parts

Commit message: Add files via upload
Parts:
- added J11, J12: Conn_01x03_Male, symbol Connector:Conn_01x03_Male
- added J13: Conn_01x02_Male, symbol Connector:Conn_01x02_Male
- gave numbers to parts that had none: 2
Connections:
- net M/IO: now reaches U7.17 (I03)
- net CLK0: no longer names the net of U8.9 (CLK0)
- net CLK0: now also J11.3 (Pin_3)
- net CLK1: no longer names the net of U8.15 (CLK1)
- net CLK1: now also J12.3 (Pin_3)
- net CLK2: no longer names the net of U8.18 (CLK2)
- net CLK2: now also J13.2 (Pin_2)
- net G0: no longer names the net of U8.11 (G0)
- net G0: now also J11.2 (Pin_2)
- net G1: no longer names the net of U8.14 (G1)
- net G1: now also J12.2 (Pin_2)
- net G2: no longer names the net of U8.16 (G2)
- net G2: now also J13.1 (Pin_1)
- net OUT0: no longer names the net of U8.10 (OUT0)
- net OUT0: now also J11.1 (Pin_1)
- net OUT1: no longer names the net of U8.13 (OUT1)
- net OUT1: now also J12.1 (Pin_1)
- no-connect marks 3 -> 2
Other:
- note added: "/O1 = A15 * A14 ... * /A5 * A4 * A3 * A2 * A1 * /A0 * M/IO"
