File: 8255x1.kicad_sch (KiCad schematic)
At the start: 6 parts

Commit message: Add files via upload
Parts:
- removed U? (x3): 74AUC2G32, symbol 74xGxx:74AUC2G32
- removed U?: 74LS04, symbol 74xx:74LS04
- added J1, J2, J3: Conn_01x08_Male, symbol Connector:Conn_01x08_Male
- gave numbers to parts that had none: 2
Connections:
- net M/IO: now also U1.17 (I03)
- net RD: now also U2.5 (~{RD})
- net WR: now also U2.36 (~{WR})
- net A15: now reaches U1.16 (IO4)
- net AD1 renamed A1
- net AD10 renamed A9
- net AD11 renamed A10
- net AD12 renamed A11
- net AD13 renamed A12
- net AD14 renamed A13
- net AD15 renamed A14
- net AD2 renamed A2
- net AD3 renamed A0
- net AD4 renamed A3
- net AD5 renamed A4
- net AD6 renamed A5
- net AD7 renamed A6
- net AD8 renamed A7
- net AD9 renamed A8
- net PA0: no longer names the net of U2.4 (PA0)
- net PA0: now also J1.8 (Pin_8)
- net PA1: no longer names the net of U2.3 (PA1)
- net PA1: now also J1.7 (Pin_7)
- net PA2: no longer names the net of U2.2 (PA2)
- net PA2: now also J1.6 (Pin_6)
- net PA3: no longer names the net of U2.1 (PA3)
- net PA3: now also J1.5 (Pin_5)
- net PA4: no longer names the net of U2.40 (PA4)
- net PA4: now also J1.4 (Pin_4)
- net PA5: no longer names the net of U2.39 (PA5)
- net PA5: now also J1.3 (Pin_3)
- net PA6: no longer names the net of U2.38 (PA6)
- net PA6: now also J1.2 (Pin_2)
- net PA7: no longer names the net of U2.37 (PA7)
- net PA7: now also J1.1 (Pin_1)
- net PB0: no longer names the net of U2.18 (PB0)
- net PB0: now also J2.8 (Pin_8)
- net PB1: no longer names the net of U2.19 (PB1)
- net PB1: now also J2.7 (Pin_7)
- net PB2: no longer names the net of U2.20 (PB2)
- net PB2: now also J2.6 (Pin_6)
- net PB3: no longer names the net of U2.21 (PB3)
- net PB3: now also J2.5 (Pin_5)
- net PB4: no longer names the net of U2.22 (PB4)
- net PB4: now also J2.4 (Pin_4)
- net PB5: no longer names the net of U2.23 (PB5)
- net PB5: now also J2.3 (Pin_3)
- net PB6: no longer names the net of U2.24 (PB6)
- net PB6: now also J2.2 (Pin_2)
- net PB7: no longer names the net of U2.25 (PB7)
- net PB7: now also J2.1 (Pin_1)
- net PC0: no longer names the net of U2.14 (PC0)
- net PC0: now also J3.8 (Pin_8)
- net PC1: no longer names the net of U2.15 (PC1)
- net PC1: now also J3.7 (Pin_7)
- net PC2: no longer names the net of U2.16 (PC2)
- net PC2: now also J3.6 (Pin_6)
- net PC3: no longer names the net of U2.17 (PC3)
- net PC3: now also J3.5 (Pin_5)
- net PC4: no longer names the net of U2.13 (PC4)
- net PC4: now also J3.4 (Pin_4)
- net PC5: no longer names the net of U2.12 (PC5)
- net PC5: now also J3.3 (Pin_3)
- net PC6: no longer names the net of U2.11 (PC6)
- net PC6: now also J3.2 (Pin_2)
- net PC7: no longer names the net of U2.10 (PC7)
- net PC7: now also J3.1 (Pin_1)
- no-connect marks 4 -> 2
Other:
- note added: "O1/ = A15 * A14 ... * M/IO"
- note removed: "Why do these OR gates have 2 extra inputs???"
