File: 8255x2.kicad_sch (KiCad schematic)
At the start: 7 parts

Commit message: Add files via upload
Parts:
- removed U? (x2): 74LS04, symbol 74xx:74LS04
- removed U?: PAL16L8, symbol Logic_Programmable:PAL16L8
- removed U? (x3): 74AUC2G32, symbol 74xGxx:74AUC2G32
- added J4, J5, J6: Conn_01x08_Male, symbol Connector:Conn_01x08_Male
- added U3: PAL16L8, symbol Logic_Programmable:PAL16L8
- gave numbers to parts that had none: 1
Connections:
- net GND: now also U3.10 (GND)
- net M/IO: now also U3.17 (I03)
- net RD: now also U4.5 (~{RD})
- net VCC: now also U3.20 (VCC)
- net WR: now also U4.36 (~{WR})
- net at U4.6 (~{CS}): now also U3.19 (IO1)
- net AD1 renamed A1
- net AD2 renamed A2
- net PA0: no longer names the net of U4.4 (PA0)
- net PA0: now also J4.8 (Pin_8)
- net PA1: no longer names the net of U4.3 (PA1)
- net PA1: now also J4.7 (Pin_7)
- net PA2: no longer names the net of U4.2 (PA2)
- net PA2: now also J4.6 (Pin_6)
- net PA3: no longer names the net of U4.1 (PA3)
- net PA3: now also J4.5 (Pin_5)
- net PA4: no longer names the net of U4.40 (PA4)
- net PA4: now also J4.4 (Pin_4)
- net PA5: no longer names the net of U4.39 (PA5)
- net PA5: now also J4.3 (Pin_3)
- net PA6: no longer names the net of U4.38 (PA6)
- net PA6: now also J4.2 (Pin_2)
- net PA7: no longer names the net of U4.37 (PA7)
- net PA7: now also J4.1 (Pin_1)
- net PB0: no longer names the net of U4.18 (PB0)
- net PB0: now also J5.8 (Pin_8)
- net PB1: no longer names the net of U4.19 (PB1)
- net PB1: now also J5.7 (Pin_7)
- net PB2: no longer names the net of U4.20 (PB2)
- net PB2: now also J5.6 (Pin_6)
- net PB3: no longer names the net of U4.21 (PB3)
- net PB3: now also J5.5 (Pin_5)
- net PB4: no longer names the net of U4.22 (PB4)
- net PB4: now also J5.4 (Pin_4)
- net PB5: no longer names the net of U4.23 (PB5)
- net PB5: now also J5.3 (Pin_3)
- net PB6: no longer names the net of U4.24 (PB6)
- net PB6: now also J5.2 (Pin_2)
- net PB7: no longer names the net of U4.25 (PB7)
- net PB7: now also J5.1 (Pin_1)
- net PC0: no longer names the net of U4.14 (PC0)
- net PC0: now also J6.8 (Pin_8)
- net PC1: no longer names the net of U4.15 (PC1)
- net PC1: now also J6.7 (Pin_7)
- net PC2: no longer names the net of U4.16 (PC2)
- net PC2: now also J6.6 (Pin_6)
- net PC3: no longer names the net of U4.17 (PC3)
- net PC3: now also J6.5 (Pin_5)
- net PC4: no longer names the net of U4.13 (PC4)
- net PC4: now also J6.4 (Pin_4)
- net PC5: no longer names the net of U4.12 (PC5)
- net PC5: now also J6.3 (Pin_3)
- net PC6: no longer names the net of U4.11 (PC6)
- net PC6: now also J6.2 (Pin_2)
- net PC7: no longer names the net of U4.10 (PC7)
- net PC7: now also J6.1 (Pin_1)
- new net A0: U3.1 (I1)
- new net A10: U3.9 (I9)
- new net A11: U3.11 (I10)
- new net A12: U3.13 (IO7)
- new net A13: U3.14 (IO6)
- new net A14: U3.15 (IO5)
- new net A15: U3.16 (IO4)
- new net A3: U3.2 (I2)
- new net A4: U3.3 (I3)
- new net A5: U3.4 (I4)
- new net A6: U3.5 (I5)
- new net A7: U3.6 (I6)
- new net A8: U3.7 (I7)
- new net A9: U3.8 (I8)
- no-connect marks 0 -> 2
Other:
- note added: "/O1 = A15 * A14 ... * /A0 * M/IO"
