File: 8259.kicad_sch (KiCad schematic)
At the start: 3 parts, among them U15 PAL16L8, U16 8259

Commit message: Add files via upload
Parts:
- added J10: Conn_01x04_Male, symbol Connector:Conn_01x04_Male
- R1: value 10000R -> 10k
Connections:
- net AD0 renamed A0
- net AD1 renamed A1
- net AD10 renamed A10
- net AD11 renamed A11
- net AD12 renamed A12
- net AD13 renamed A13
- net AD14 renamed A14
- net AD15 renamed A15
- net AD2 renamed A2
- net AD3 renamed A3
- net AD4 renamed A4
- net AD5 renamed A5
- net AD6 renamed A6
- net AD7 renamed A7
- net AD8 renamed A8
- net AD9 renamed A9
- net IORC renamed RD
- net IOWC renamed WR
- net IR4: no longer names the net of U16.22 (IR4)
- net IR4: now also J10.1 (Pin_1)
- net IR5: no longer names the net of U16.23 (IR5)
- net IR5: now also J10.2 (Pin_2)
- net IR6: no longer names the net of U16.24 (IR6)
- net IR6: now also J10.3 (Pin_3)
- net IR7: no longer names the net of U16.25 (IR7)
- net IR7: now also J10.4 (Pin_4)
Other:
- note added: "/O1 = A15 * A14 ... * A4 * /A3 * A2 * A1 * /A0"
- note added: "SP high to designate as master"
- moved on the sheet: R1
