File: 8279.kicad_sch (KiCad schematic)
At the start: 28 parts

Commit message: Add files via upload
Parts:
- added R2: 10k, symbol Device:R
- gave numbers to parts that had none: 28
Connections:
- net GND: now also U11.4 (E1), U11.5 (E2), U11.8 (GND)
- net VCC: now also U11.16 (VCC), R2.2
- net at SW11.2, SW12.2, SW13.2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: now also U11.13 (O2)
- net at U11.1 (A0): now also U9.32 (SL0)
- net at U11.11 (O4): now also SW21.2, SW22.2, SW23.2, SW24.2, SW25.2
- net at U11.12 (O3): now also SW16.2, SW17.2, SW18.2, SW19.2, SW20.2
- net at U11.14 (O1): now also SW10.2, SW6.2, SW7.2, SW8.2, SW9.2
- net at U11.15 (O0): now also SW1.2, SW2.2, SW3.2, SW4.2, SW5.2
- net at U11.2 (A1): now also U9.33 (SL1)
- net at U11.3 (A2): now also U9.34 (SL2)
- net at U11.6 (E3): now also R2.1
- net AD0 renamed A0
- net AD1 renamed A1
- net AD10 renamed A10
- net AD11 renamed A11
- net AD12 renamed A12
- net AD13 renamed A13
- net AD14 renamed A14
- net AD15 renamed A15
- net AD2 renamed A2
- net AD3 renamed A3
- net AD4 renamed A4
- net AD5 renamed A5
- net AD6 renamed A6
- net AD7 renamed A7
- net AD8 renamed A8
- net AD9 renamed A9
- no-connect marks 6 -> 10
Other:
- note added: "/O1 = A15 * A14...... * A4 * /A3 * /A2 * A1 * /A0"
- note added: "IRQ outputs to 8259"
